File: PCB/Serial-TTL-Converter.kicad_pcb (KiCad board)
At the start: 2 copper layers, 68 parts, among them J1 RS232 (PC), J2 TTL (uC), J3 power-supply, Q1 BC817, Q2 BC817, Q3 BC817, Q4 BC817, Q5 BC817, Q6 BC817, SW1 SW_SPDT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

Commit message: PCB routing
Parts:
- added C12: 100u/6V3, Capacitor_THT:CP_Radial_D6.3mm_P2.50mm, B.Cu at (67.0, 55.9)
- C1: value 1u -> 100u/6V3; footprint Capacitors_Tantalum_SMD:CP_Tantalum_Case-C_EIA-6032-28_Reflow -> Capacitor_THT:CP_Radial_D6.3mm_P2.50mm; moved to B.Cu
- C10: value 160u -> 270u/16V; footprint Capacitor_THT:CP_Radial_D6.3mm_P2.50mm -> Capacitor_THT:CP_Radial_D8.0mm_P3.50mm; moved to B.Cu
- C11: value 100n -> 1u
- C12, U3: moved to B.Cu
- C6: value 1u -> 100u/6V3; footprint Capacitors_SMD:C_0805 -> Capacitor_THT:CP_Radial_D6.3mm_P2.50mm
- C7: value 160u -> 100n; footprint Capacitor_THT:CP_Radial_Tantal_D6.0mm_P2.50mm -> Capacitors_SMD:C_0805
- moved SW1 187.9 mm to (81.1, 54.7)
- moved U4 185.5 mm to (67.8, 39.7), turned to 90 degrees
- moved C12 177.2 mm to (64.7, 49.1), turned to 90 degrees
- moved C11 174.5 mm to (70.1, 47.5), turned to 90 degrees
- moved D9 173.8 mm to (90.7, 41.7)
- moved F2 173.8 mm to (87.4, 47.3)
- moved F3 173.8 mm to (80.6, 46.8)
- moved J3 173.8 mm to (80.6, 40.7)
- moved C10 92.0 mm to (130.7, 63.4), turned to 90 degrees
- moved D7 79.1 mm to (127.1, 53.3), turned to 270 degrees
- moved D8 75.1 mm to (141.3, 63.0), turned to 180 degrees
- moved R22 73.8 mm to (134.0, 57.5), turned to 270 degrees
- moved C7 72.2 mm to (137.3, 40.6), turned to 90 degrees
- moved L2 63.1 mm to (132.5, 53.0), turned to 270 degrees
- moved C6 55.1 mm to (131.4, 43.9), turned to 90 degrees
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Connections:
- C10 pad 1: -12V -> GND
- C10 pad 2: GND -> -12V
- J1 pad 2: /RTS -> /RI
- J1 pad 3: /DTR -> /RTS
- J1 pad 4: /TX -> /CTS
- J1 pad 5: /RI -> /DTR
- J1 pad 6: /CTS -> /TX
Routing:
- net +5V: track 0.00 -> 80.4 mm
- net Net-(D2-Pad1): track 0.00 -> 18.6 mm
- net Net-(D3-Pad1): track 0.00 -> 17.3 mm
- net Net-(D4-Pad1): track 0.00 -> 15.0 mm
- net Net-(D5-Pad1): track 0.00 -> 14.8 mm
- net -12V: track 0.00 -> 14.4 mm
- net Net-(D7-Pad1): track 0.00 -> 12.9 mm
- net /DCD: track 0.00 -> 12.1 mm
- net Net-(D8-Pad2): track 0.00 -> 12.1 mm
- net Net-(D6-Pad1): track 0.00 -> 11.7 mm
- net /RX: track 0.00 -> 11.6 mm
- net /RI: track 0.00 -> 11.5 mm
- net /DSR: track 0.00 -> 11.1 mm
- net /RTS: track 0.00 -> 11.0 mm
- net /TX: track 0.00 -> 10.6 mm
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Other:
- net class Default: clearance 0.2 -> 0.7
- rule trace_clearance: 0.2 -> 0.7

Commit message: PCB routing
Parts:
- moved F1 46.7 mm to (93.7, 85.2), turned to 90 degrees
- moved U4 38.9 mm to (101.4, 59.1)
- moved C12 36.3 mm to (101.3, 67.7), turned to 180 degrees
- moved SW1 15.1 mm to (87.7, 68.2), turned to 180 degrees
- moved C5 9.13 mm to (105.9, 53.8)
- moved C10 7.87 mm to (123.9, 59.4), turned to 0 degrees
- moved R18 7.69 mm to (136.7, 68.4), turned to 0 degrees
- moved D5 7.47 mm to (126.7, 66.1), turned to 180 degrees
- moved R17 7.29 mm to (126.1, 68.2), turned to 180 degrees
- moved C14 6.36 mm to (127.4, 87.4)
- moved C13 6.36 mm to (128.4, 72.3)
- moved D3 6.36 mm to (139.3, 92.5)
- moved D4 6.36 mm to (139.3, 88.7)
- moved J1 6.36 mm to (107.9, 68.8)
- moved J2 6.36 mm to (129.5, 96.3)
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Connections:
- J2 pad 1: Net-(F1-Pad1) -> /DCD_UC
- J2 pad 10: GND -> Net-(F1-Pad1)
- J2 pad 3: /CTS_UC -> /DSR_UC
- J2 pad 4: /DCD_UC -> /TX_UC
- J2 pad 5: /DSR_UC -> /DTR_UC
- J2 pad 6: /DTR_UC -> /RTS_UC
- J2 pad 7: /RI_UC -> /CTS_UC
- J2 pad 8: /TX_UC -> /RI_UC
- J2 pad 9: /RTS_UC -> GND
Routing:
- net /RTS_UC: track 3.26 -> 67.7 mm
- net /DTR_UC: track 2.81 -> 53.2 mm
- net +5V: track 80.4 -> 118.4 mm
- net /TX_UC: track 2.92 -> 40.1 mm
- net /CTS_UC: track 0.00 -> 37.1 mm
- net GND: track 1.89 -> 20.5 mm, vias 0 -> 4
- net VCC: track 8.90 -> 25.1 mm, vias 0 -> 3
- net -12V: track 14.4 -> 28.9 mm
- net /RI_UC: track 0.00 -> 13.8 mm
- net /DCD_UC: track 0.00 -> 6.18 mm
- net Net-(D1-Pad2): track 8.33 -> 6.40 mm
- net Net-(D6-Pad1): track 11.7 -> 13.1 mm

Commit message: PCB routing
Parts:
- removed the C12 at (64.7, 49.1)
- moved C11 42.8 mm to (108.4, 66.4), turned to 0 degrees
- moved J3 42.6 mm to (98.6, 79.2)
- moved F3 31.7 mm to (98.7, 72.8), turned to 270 degrees
- moved F2 30.1 mm to (103.2, 72.9), turned to 270 degrees
- moved SW1 27.5 mm to (101.3, 92.2), turned to 0 degrees
- moved D9 24.4 mm to (100.7, 64.0), turned to 180 degrees
- moved F1 18.8 mm to (104.5, 100.6), turned to 180 degrees
- moved C5 10.3 mm to (116.2, 53.5), turned to 90 degrees
- moved U4 9.42 mm to (110.5, 61.8), turned to 0 degrees
- moved C12 7.41 mm to (103.2, 60.6), turned to 90 degrees
- moved R8 0.47 mm to (112.7, 43.3)
Connections:
- U3 pad 7: Net-(U3-Pad7) -> (no net)
Routing:
- net +5V: track 118.4 -> 145.1 mm
- net Net-(D9-Pad2): track 0.00 -> 11.2 mm
- net Net-(F3-Pad2): track 0.00 -> 5.35 mm
- net +3V3: track 0.00 -> 4.62 mm
- net Net-(F2-Pad2): track 0.00 -> 4.42 mm
- net Net-(D1-Pad2): track 6.40 -> 9.51 mm
Other:
- board outline added: 61 x 68.9 mm

Commit message: PCB routing
Parts:
- moved SW1 1.38 mm to (101.4, 90.8)
- moved D8 0.32 mm to (141.5, 62.7)
- moved D3 0.20 mm to (139.3, 92.7)
- moved D4 0.20 mm to (139.3, 88.5)
Routing:
- net VCC: track 25.1 -> 98.6 mm, vias 3 -> 4
- net +12V: track 1.22 -> 62.9 mm, vias 0 -> 3
- net /RI_UC: track 13.8 -> 51.9 mm, vias 0 -> 1
- net +3V3: track 4.62 -> 40.8 mm, vias 0 -> 1
- net /DSR_UC: track 0.00 -> 19.2 mm, vias 0 -> 2
- net +5V: track 145.1 -> 163.8 mm
- net /RX_UC: track 0.00 -> 11.6 mm, vias 0 -> 2
- net GND: track 20.5 -> 29.1 mm, vias 4 -> 8
- net Net-(F1-Pad1): track 0.00 -> 4.29 mm
- net -12V: track 28.9 -> 33.0 mm
