File: PCB/Serial-TTL-Converter.sch (KiCad schematic (older format))
At the start: 71 parts

Commit message: Add footprints, remove TTL inputs transistors, add 3V3 supply
Parts:
- removed Q? (x10): BC817, TO_SOT_Packages_SMD:SOT-23, symbol Transistor_BJT:BC817
- removed R? (x5): 4k7, Resistors_SMD:R_0805, symbol Device:R
- removed R? (x15): 10k, Resistors_SMD:R_0805, symbol Device:R
- removed R? (x5): 2k2, Resistors_SMD:R_0805, symbol Device:R
- added C? (x5): 100n, Capacitors_SMD:C_0805, symbol Device:C
- added C? (x2): 22u, symbol Device:CP
- added C?: 1u, symbol Device:CP
- added C?: 160u, symbol Device:CP
- added C?: 1u, Capacitors_SMD:C_0805, symbol Device:CP
- added C?: 160u, symbol Device:C
- added D? (x2): D_Schottky, symbol Device:D_Schottky
- added D? (x5): 5V1, symbol Device:D_Zener
- added F? (x2): 500mA, symbol Device:Fuse
- added F?: Fuse, symbol Device:Fuse
- added J?: power-supply, symbol Connector_Generic:Conn_01x03
- added L?: LPS4018-103 (10uH), Inductor_SMD:L_Coilcraft_LPS4018, symbol Device:L
- added R?: 10k, Resistors_SMD:R_0805, symbol Device:R
- added R? (x5): 330R, Resistors_SMD:R_0805, symbol Device:R
- added SW?: SW_SPDT, symbol Switch:SW_SPDT
- added U?: AP1117-33, TO_SOT_Packages_SMD:SOT-223, symbol Regulator_Linear:AP1117-33
- C?: value C -> 100n; footprint (none) -> Capacitors_SMD:C_0805
- C?: value C -> 2n2; footprint (none) -> Capacitors_SMD:C_0805
- C?: value C -> 47p; footprint (none) -> Capacitors_SMD:C_0805
- C?: value C -> 2u2; footprint (none) -> Capacitors_SMD:C_0805
- L?: value L -> LPS4018-223 (22uH); footprint (none) -> Inductor_SMD:L_Coilcraft_LPS4018
- R?: value 10k -> 56k
- R?: value 10k -> 6.2k
- R?: value 10k -> 130k
- U?: footprint (none) -> Housings_SOIC:SO-20_12.8x7.5mm_Pitch1.27mm
- U?: footprint (none) -> Housings_SSOP:MSOP-8-1EP_3x3mm_Pitch0.65mm
Connections:
- net +12V: now also C?.1
- net +5V: now also U?.1 (V+), U?.13 (V+), U?.14 (V+), U?.2 (/SHDN), C?.1, C?.1, C?.1, C?.1, C?.1, F?.1, F?.1, SW?.3 (C), U?.3 (VI); no longer R?.2, R?.2, R?.2, R?.2, R?.2, R?.2
- net -12V: now also U?.8 (VOUT), C?.1, C?.1, D?.2 (A), R?.2
- net CTS_L: no longer U?.7 (RA4)
- net CTS_UC: now also R?.2
- net DCD_UC: now also R?.2
- net DSR_UC: now also R?.2
- net GND: now also C?.2, C?.2, C?.2, C?.2, C?.2, C?.2, C?.2, C?.2, C?.2, C?.2, C?.2, D?.1 (K), D?.2 (A), D?.2 (A), D?.2 (A), D?.2 (A), D?.2 (A), J?.1 (Pin_1), L?.2, U?.1 (GND)
- net RI_UC: now also R?.2
- net RX_UC: now also R?.2
- net VCC: now also R?.2, R?.2, R?.2, R?.2, R?.2, R?.2, F?.2, SW?.2 (B); no longer J?.1 (Pin_1)
- net at U?.11 (LX): now also U?.12 (LX), D?.1 (K), L?.1
- net at U?.3 (VREF): now also C?.1
- net at U?.5 (SS): now also C?.1
- net at U?.9 (DRV-): now also D?.2 (A), R?.1
- net DCD_L: no longer names the net of U?.2 (RA1)
- net DCD_L: now also D?.1 (K), R?.1
- net DSR_L: no longer names the net of U?.4 (RA3)
- net DSR_L: now also D?.1 (K), R?.1
- net RI_L: no longer names the net of U?.9 (RA5)
- net RI_L: now also D?.1 (K), R?.1
- net RX_L: no longer names the net of U?.3 (RA2)
- net RX_L: now also D?.1 (K), R?.1
- new net: D?.1 (K), R?.1, U?.7 (RA4)
- new net: F?.1, J?.1 (Pin_1)
- new net: F?.2, J?.2 (Pin_2)
- new net: F?.2, J?.3 (Pin_3)
- new net +3V3: C?.1, SW?.1 (A), U?.2 (VO)
Other:
- note added: "3V3 LDO regulator"
- note added: "3V3/5V power supply switch\n"
- note added: "5V -> -12V converter"
- note added: "5V -> 12V converter"
- note added: "5x330R\n"
- note added: "5x5V1"
- note added: "Power supply input connector\n"
- note added: "RS232 <-> TTL converter"
- moved on the sheet: C?, D?, J?, L?, Q?, R?, U?

Commit message: Footprints update, PCB routing
Parts:
- removed F? (x2): 500mA, symbol Device:Fuse
- added D9: STPS1L30U, Diodes_SMD:D_SMB, symbol Device:D_Schottky
- added F2, F3: 500mA (SD050-16 ECE), Fuse:Fuse_1812_4532Metric, symbol Device:Fuse
- C1, C8: renamed from C?; footprint (none) -> Capacitors_Tantalum_SMD:CP_Tantalum_Case-C_EIA-6032-28_Reflow
- C10: renamed from C?; footprint (none) -> Capacitor_THT:CP_Radial_D6.3mm_P2.50mm
- C12: renamed from C?; footprint (none) -> Capacitor_THT:CP_Radial_D5.0mm_P2.50mm
- C7: renamed from C?; footprint (none) -> Capacitor_THT:CP_Radial_Tantal_D6.0mm_P2.50mm
- D1, D7, D8: renamed from D?; value D_Schottky -> STPS1L30U; footprint (none) -> Diodes_SMD:D_SMB
- D2, D3, D4, D5, D6: renamed from D?; footprint (none) -> Diodes_SMD:D_MiniMELF
- F1: renamed from F?; value Fuse -> 500mA (SD050-16 ECE); footprint (none) -> Fuse:Fuse_1812_4532Metric
- J1: renamed from J?; footprint (none) -> Connectors:1X09_LONGPADS
- J2: renamed from J?; footprint (none) -> Connector_PinHeader_2.54mm:PinHeader_1x10_P2.54mm_Vertical
- J3: renamed from J?; footprint (none) -> Connectors:1X03_LONGPADS
- SW1: renamed from SW?; footprint (none) -> Switches:SWITCH_SPDT_PTH_11.6X4.0MM
- U3: renamed from U?; footprint (none) -> Silicon-Standard:DIP14
- gave numbers to parts that had none: 46
Connections:
- net CTS_L is gone; now on net RTS_L: R20.1
- net +12V: no longer U1.4 (SW)
- net +5V: now also D9.1 (K)
- net CTS_UC: no longer Q6.3 (C), R25.1
- net RTS_UC: now also Q6.3 (C), R25.1
- net at D1.2 (A), L1.2: now also U1.4 (SW)
- net at J3.2 (Pin_2): now also F3.2
- net at J3.3 (Pin_3): now also F2.2
- new net: D9.2 (A), F2.1, F3.1
Other:
- moved on the sheet: D1

Commit message: Capacitor footprint change
Parts:
- removed C12: 22u, Capacitor_THT:CP_Radial_D5.0mm_P2.50mm, symbol Device:CP
- added C?: 100u/6V3, Capacitor_THT:CP_Radial_D6.3mm_P2.50mm, symbol Device:CP
- C1: value 1u -> 100u/6V3; footprint Capacitors_Tantalum_SMD:CP_Tantalum_Case-C_EIA-6032-28_Reflow -> Capacitor_THT:CP_Radial_D6.3mm_P2.50mm
- C10: value 160u -> 270u/16V; footprint Capacitor_THT:CP_Radial_D6.3mm_P2.50mm -> Capacitor_THT:CP_Radial_D8.0mm_P3.50mm
- C11: value 100n -> 1u
- C6: value 1u -> 100u/6V3; footprint Capacitors_SMD:C_0805 -> Capacitor_THT:CP_Radial_D6.3mm_P2.50mm
- C7: value 160u -> 100n; footprint Capacitor_THT:CP_Radial_Tantal_D6.0mm_P2.50mm -> Capacitors_SMD:C_0805
- U1: symbol project-symbols:LT8570 -> Serial-TTL-Converter-rescue:LT8570-project-symbols
- U2: symbol project-symbols:ST75185 -> Serial-TTL-Converter-rescue:ST75185-project-symbols
- U3: symbol project-symbols:MAX736 -> Serial-TTL-Converter-rescue:MAX736-project-symbols
Connections:
- net +3V3: now also C?.1
- net -12V: now also C10.2; no longer C10.1
- net GND: now also C10.1, C?.2; no longer C10.2
Changed lines of the file:
@@
 $EndDescr
 $Comp
-L project-symbols:ST75185 U2
+L Serial-TTL-Converter-rescue:ST75185-project-symbols U2
 U 1 1 5F215863
 P 5100 4850
@@
 $EndComp
 $Comp
-L project-symbols:LT8570 U1
+L Serial-TTL-Converter-rescue:LT8570-project-symbols U1
 U 1 1 5F2172C9
 P 3150 2700
@@
 P 2300 3100
 F 0 "C1" H 2418 3146 50  0000 L CNN
-F 1 "1u" H 2418 3055 50  0000 L CNN
-F 2 "Capacitors_Tantalum_SMD:CP_Tantalum_Case-C_EIA-6032-28_Reflow" H 2338 2950 50  0001 C CNN
+F 1 "100u/6V3" H 2418 3055 50  0000 L CNN
+F 2 "Capacitor_THT:CP_Radial_D6.3mm_P2.50mm" H 2338 2950 50  0001 C CNN
 F 3 "~" H 2300 3100 50  0001 C CNN
 	1    2300 3100
@@
 P 10300 2900
 F 0 "C11" H 10100 2950 50  0000 L CNN
-F 1 "100n" H 10000 2850 50  0000 L CNN
+F 1 "1u" H 10000 2850 50  0000 L CNN
 F 2 "Capacitors_SMD:C_0805" H 10338 2750 50  0001 C CNN
 F 3 "~" H 10300 2900 50  0001 C CNN
@@
 Wire Wire Line
 	11250 3100 11250 3050
-$Comp
-L Device:CP C12
-U 1 1 5F56E50A
-P 11250 2900
-F 0 "C12" H 11368 2946 50  0000 L CNN
-F 1 "22u" H 11368 2855 50  0000 L CNN
-F 2 "Capacitor_THT:CP_Radial_D5.0mm_P2.50mm" H 11288 2750 50  0001 C CNN
-F 3 "~" H 11250 2900 50  0001 C CNN
-	1    11250 2900
-	1    0    0    -1
-$EndComp
 Wire Wire Line
 	10750 3250 10750 3100
@@
 P 5650 3150
 F 0 "C7" H 5765 3196 50  0000 L CNN
-F 1 "160u" H 5765 3105 50  0000 L CNN
-F 2 "Capacitor_THT:CP_Radial_Tantal_D6.0mm_P2.50mm" H 5688 3000 50  0001 C CNN
+F 1 "100n" H 5765 3105 50  0000 L CNN
+F 2 "Capacitors_SMD:C_0805" H 5688 3000 50  0001 C CNN
 F 3 "~" H 5650 3150 50  0001 C CNN
 	1    5650 3150
 	1    0    0    -1
 $EndComp
-$Comp
-L Device:CP C6
-U 1 1 5F576334
-P 5300 3150
-F 0 "C6" H 5418 3196 50  0000 L CNN
-F 1 "1u" H 5418 3105 50  0000 L CNN
-F 2 "Capacitors_SMD:C_0805" H 5338 3000 50  0001 C CNN
-F 3 "~" H 5300 3150 50  0001 C CNN
-	1    5300 3150
-	1    0    0    -1
-$EndComp
 Connection ~ 8750 3200
 Wire Wire Line
@@
 Wire Wire Line
 	8750 2450 9100 2450
-$Comp
-L Device:CP C10
-U 1 1 5F5464C8
-P 9100 2600
-F 0 "C10" H 9218 2646 50  0000 L CNN
-F 1 "160u" H 9218 2555 50  0000 L CNN
-F 2 "Capacitor_THT:CP_Radial_D6.3mm_P2.50mm" H 9138 2450 50  0001 C CNN
-F 3 "~" H 9100 2600 50  0001 C CNN
-	1    9100 2600
-	1    0    0    -1
-$EndComp
 Wire Wire Line
 	8400 2450 8750 2450
@@
 	1    8750 3200
 	1    0    0    -1
-$EndComp
-$Comp
-L Device:R R22
-U 1 1 5F3F9894
-P 8750 2600
-F 0 "R22" H 8850 2570 50  0000 C CNN
-F 1 "10k" H 8870 2640 50  0000 C CNN
-F 2 "Resistors_SMD:R_0805" V 8680 2600 50  0001 C CNN
-F 3 "~" H 8750 2600 50  0001 C CNN
-	1    8750 2600
-	1    0    0    1
 $EndComp
 $Comp
@@
 	6750 3150 6800 3150
 $Comp
-L project-symbols:MAX736 U3
+L Serial-TTL-Converter-rescue:MAX736-project-symbols U3
 U 1 1 5F217A34
 P 6900 2400
@@
 Wire Wire Line
 	3450 2400 3900 2400
+$Comp
+L Device:CP C10
+U 1 1 5F5464C8
+P 9100 2600
+F 0 "C10" H 8750 2550 50  0000 L CNN
+F 1 "270u/16V" H 8600 2650 50  0000 L CNN
+F 2 "Capacitor_THT:CP_Radial_D8.0mm_P3.50mm" H 9138 2450 50  0001 C CNN
+F 3 "~" H 9100 2600 50  0001 C CNN
+	1    9100 2600
+	-1   0    0    1
+$EndComp
+$Comp
+L Device:R R22
+U 1 1 5F3F9894
+P 8750 2600
+F 0 "R22" H 8850 2570 50  0000 C CNN
+F 1 "10k" H 8850 2650 50  0000 C CNN
+F 2 "Resistors_SMD:R_0805" V 8680 2600 50  0001 C CNN
+F 3 "~" H 8750 2600 50  0001 C CNN
+	1    8750 2600
+	1    0    0    1
+$EndComp
+$Comp
+L Device:CP C?
+U 1 1 5F3EFCCE
+P 11250 2900
+F 0 "C?" H 11368 2946 50  0000 L CNN
+F 1 "100u/6V3" H 11368 2855 50  0000 L CNN
+F 2 "Capacitor_THT:CP_Radial_D6.3mm_P2.50mm" H 11288 2750 50  0001 C CNN
+F 3 "~" H 11250 2900 50  0001 C CNN
+	1    11250 2900
+	1    0    0    -1
+$EndComp
+$Comp
+L Device:CP C6
+U 1 1 5F576334
+P 5300 3150
+F 0 "C6" H 5418 3196 50  0000 L CNN
+F 1 "100u/6V3" H 5350 3050 35  0000 L CNN
+F 2 "Capacitor_THT:CP_Radial_D6.3mm_P2.50mm" H 5338 3000 35  0001 C CNN
+F 3 "~" H 5300 3150 50  0001 C CNN
+	1    5300 3150
+	1    0    0    -1
+$EndComp
 $EndSCHEMATC

Commit message: PCB routing
Parts:
- gave numbers to parts that had none: 1
Connections:
- net CTS: now also J1.4 (Pin_4); no longer J1.6 (Pin_6)
- net DTR: now also J1.5 (Pin_5); no longer J1.3 (Pin_3)
- net RI: now also J1.2 (Pin_2); no longer J1.5 (Pin_5)
- net RTS: now also J1.3 (Pin_3); no longer J1.2 (Pin_2)
- net TX: now also J1.6 (Pin_6); no longer J1.4 (Pin_4)
Changed lines of the file:
@@
 	4250 5200 2850 5200
 Wire Wire Line
-	4250 5300 2850 5300
-Wire Wire Line
-	4250 5400 2850 5400
-Wire Wire Line
 	4250 5550 3500 5550
 Wire Wire Line
-	3500 5550 3500 5500
-Wire Wire Line
-	3500 5500 2850 5500
-Wire Wire Line
 	4250 5650 3400 5650
 Wire Wire Line
 	3400 5650 3400 5600
-Wire Wire Line
-	3400 5600 2850 5600
-Wire Wire Line
-	4250 5750 3350 5750
-Wire Wire Line
-	3350 5750 3350 5700
-Wire Wire Line
-	3350 5700 2850 5700
 $Comp
 L power:GND #PWR0105
@@
 Text Label 3100 5200 0    50   ~ 0
 DSR
-Text Label 3100 5300 0    50   ~ 0
+Text Label 3400 5300 0    50   ~ 0
 CTS
-Text Label 3100 5400 0    50   ~ 0
-RI
-Text Label 3100 5500 0    50   ~ 0
+Text Label 3600 5550 0    50   ~ 0
 TX
-Text Label 3100 5600 0    50   ~ 0
+Text Label 3500 5650 0    50   ~ 0
 DTR
-Text Label 3100 5700 0    50   ~ 0
-RTS
 Text Label 5700 5550 2    50   ~ 0
 TX_L
@@
 $EndComp
 $Comp
-L Device:CP C?
+L Device:CP C12
 U 1 1 5F3EFCCE
 P 11250 2900
-F 0 "C?" H 11368 2946 50  0000 L CNN
+F 0 "C12" H 11368 2946 50  0000 L CNN
 F 1 "100u/6V3" H 11368 2855 50  0000 L CNN
 F 2 "Capacitor_THT:CP_Radial_D6.3mm_P2.50mm" H 11288 2750 50  0001 C CNN
@@
 	1    0    0    -1
 $EndComp
+Text Label 3100 5700 0    50   ~ 0
+RI
+Text Label 3500 5750 0    50   ~ 0
+RTS
+Wire Wire Line
+	4250 5400 3250 5400
+Wire Wire Line
+	3250 5400 3250 5700
+Wire Wire Line
+	3250 5700 2850 5700
+Wire Wire Line
+	3000 5750 4250 5750
+Wire Wire Line
+	2850 5600 3000 5600
+Wire Wire Line
+	3000 5600 3000 5750
+Wire Wire Line
+	3050 5300 3050 5500
+Wire Wire Line
+	3050 5500 2850 5500
+Wire Wire Line
+	3050 5300 4250 5300
+Wire Wire Line
+	2850 5400 3150 5400
+Wire Wire Line
+	3150 5400 3150 5600
+Wire Wire Line
+	3150 5600 3400 5600
+Wire Wire Line
+	2850 5300 2950 5300
+Wire Wire Line
+	2950 5300 2950 5350
+Wire Wire Line
+	2950 5350 3500 5350
+Wire Wire Line
+	3500 5350 3500 5550
 $EndSCHEMATC

Commit message: PCB routing
Connections:
- net CTS_UC: now also J2.7 (Pin_7); no longer J2.3 (Pin_3)
- net DCD_UC: now also J2.1 (Pin_1); no longer J2.4 (Pin_4)
- net DSR_UC: now also J2.3 (Pin_3); no longer J2.5 (Pin_5)
- net DTR_UC: now also J2.5 (Pin_5); no longer J2.6 (Pin_6)
- net GND: now also J2.9 (Pin_9); no longer J2.10 (Pin_10)
- net RI_UC: now also J2.8 (Pin_8); no longer J2.7 (Pin_7)
- net RTS_UC: now also J2.6 (Pin_6); no longer J2.9 (Pin_9)
- net TX_UC: now also J2.4 (Pin_4); no longer J2.8 (Pin_8)
- net at F1.1: now also J2.10 (Pin_10); no longer J2.1 (Pin_1)
Other:
- moved on the sheet: F1, J2
Changed lines of the file:
@@
 L Connector_Generic:Conn_01x10 J2
 U 1 1 5F3A338E
-P 9250 5450
-F 0 "J2" H 9330 5442 50  0000 L CNN
-F 1 "TTL (uC)" H 9330 5351 50  0000 L CNN
-F 2 "Connector_PinHeader_2.54mm:PinHeader_1x10_P2.54mm_Vertical" H 9250 5450 50  0001 C CNN
-F 3 "~" H 9250 5450 50  0001 C CNN
-	1    9250 5450
-	1    0    0    -1
-$EndComp
-Wire Wire Line
-	9050 5150 8350 5150
-Wire Wire Line
-	9050 5250 8350 5250
-Wire Wire Line
-	9050 5350 8350 5350
-Wire Wire Line
-	9050 5450 8350 5450
-Wire Wire Line
-	9050 5550 8350 5550
-Wire Wire Line
-	9050 5650 8350 5650
-Wire Wire Line
-	9050 5750 8350 5750
-Wire Wire Line
-	9050 5850 8350 5850
+P 9550 5550
+F 0 "J2" H 9630 5542 50  0000 L CNN
+F 1 "TTL (uC)" H 9630 5451 50  0000 L CNN
+F 2 "Connector_PinHeader_2.54mm:PinHeader_1x10_P2.54mm_Vertical" H 9550 5550 50  0001 C CNN
+F 3 "~" H 9550 5550 50  0001 C CNN
+	1    9550 5550
+	1    0    0    1
+$EndComp
 $Comp
 L power:GND #PWR0112
 U 1 1 5F2A03D4
-P 9000 6050
-F 0 "#PWR0112" H 9000 5800 50  0001 C CNN
-F 1 "GND" H 9005 5877 50  0000 C CNN
-F 2 "" H 9000 6050 50  0001 C CNN
-F 3 "" H 9000 6050 50  0001 C CNN
-	1    9000 6050
+P 9000 6250
+F 0 "#PWR0112" H 9000 6000 50  0001 C CNN
+F 1 "GND" H 9005 6077 50  0000 C CNN
+F 2 "" H 9000 6250 50  0001 C CNN
+F 3 "" H 9000 6250 50  0001 C CNN
+	1    9000 6250
 	-1   0    0    -1
 $EndComp
 Wire Wire Line
-	9000 6050 9000 5950
-Wire Wire Line
-	9000 5950 9050 5950
+	9000 6250 9000 5150
 Text Label 4900 7450 2    50   ~ 0
 TX_UC
 Text Label 10150 7500 2    50   ~ 0
 RTS_UC
-Text Label 8350 5150 0    50   ~ 0
-RX_UC
-Text Label 8350 5250 0    50   ~ 0
-CTS_UC
-Text Label 8350 5350 0    50   ~ 0
-DCD_UC
-Text Label 8350 5450 0    50   ~ 0
-DSR_UC
-Text Label 8350 5550 0    50   ~ 0
-DTR_UC
-Text Label 8350 5650 0    50   ~ 0
-RI_UC
-Text Label 8350 5750 0    50   ~ 0
-TX_UC
-Text Label 8350 5850 0    50   ~ 0
-RTS_UC
 $Comp
 L power:VCC #PWR0113
 U 1 1 5F2D1E1B
-P 8700 4900
-F 0 "#PWR0113" H 8700 4750 50  0001 C CNN
-F 1 "VCC" H 8717 5073 50  0000 C CNN
-F 2 "" H 8700 4900 50  0001 C CNN
-F 3 "" H 8700 4900 50  0001 C CNN
-	1    8700 4900
-	1    0    0    -1
-$EndComp
-Wire Wire Line
-	9050 5050 9000 5050
-Wire Wire Line
-	8700 5050 8700 4900
+P 9000 4900
+F 0 "#PWR0113" H 9000 4750 50  0001 C CNN
+F 1 "VCC" H 9017 5073 50  0000 C CNN
+F 2 "" H 9000 4900 50  0001 C CNN
+F 3 "" H 9000 4900 50  0001 C CNN
+	1    9000 4900
+	1    0    0    -1
+$EndComp
+Wire Wire Line
+	9350 5050 9300 5050
+Wire Wire Line
+	9000 5050 9000 4900
 $Comp
 L power:+5V #PWR0114
@@
 L Device:Fuse F1
 U 1 1 5F6E306A
-P 8850 5050
-F 0 "F1" V 8653 5050 50  0000 C CNN
-F 1 "500mA (SD050-16 ECE)" V 8744 5050 50  0000 C CNN
-F 2 "Fuse:Fuse_1812_4532Metric" V 8780 5050 50  0001 C CNN
-F 3 "~" H 8850 5050 50  0001 C CNN
-	1    8850 5050
+P 9150 5050
+F 0 "F1" V 8953 5050 50  0000 C CNN
+F 1 "500mA (SD050-16 ECE)" V 9044 5050 50  0000 C CNN
+F 2 "Fuse:Fuse_1812_4532Metric" V 9080 5050 50  0001 C CNN
+F 3 "~" H 9150 5050 50  0001 C CNN
+	1    9150 5050
 	0    1    1    0
 $EndComp
@@
 Wire Wire Line
 	3500 5350 3500 5550
+Wire Wire Line
+	9000 5150 9350 5150
+Wire Wire Line
+	9350 5850 8650 5850
+Wire Wire Line
+	9350 5350 8650 5350
+Wire Wire Line
+	9350 5950 8650 5950
+Wire Wire Line
+	9350 5750 8650 5750
+Wire Wire Line
+	9350 5550 8650 5550
+Wire Wire Line
+	9350 5250 8650 5250
+Wire Wire Line
+	9350 5650 8650 5650
+Wire Wire Line
+	9350 5450 8650 5450
+Text Label 8650 5850 0    50   ~ 0
+RX_UC
+Text Label 8650 5350 0    50   ~ 0
+CTS_UC
+Text Label 8650 5950 0    50   ~ 0
+DCD_UC
+Text Label 8650 5750 0    50   ~ 0
+DSR_UC
+Text Label 8650 5550 0    50   ~ 0
+DTR_UC
+Text Label 8650 5250 0    50   ~ 0
+RI_UC
+Text Label 8650 5650 0    50   ~ 0
+TX_UC
+Text Label 8650 5450 0    50   ~ 0
+RTS_UC
 $EndSCHEMATC
